Commit message: Added camera link

File: config/robot/urdf/ardent.urdf.xacro (robot description, xacro)
@@ -5,6 +5,44 @@
 <!-- =================================================================================== -->
 <robot name="ardent" xmlns:xacro="http://www.ros.org/wiki/xacro">
-  <!-- <xacro:property name="joint_effort" value ="10000"/>
-<xacro:property name="joint_velocity" value ="100"/> -->
+  <!-- Size of square 'camera' box -->
+  <!-- Link-->
+  <joint name="camera_joint" type="fixed">
+    <axis xyz="0 1 0"/>
+    <origin rpy="0 0 0" xyz="0.2 0 0"/>
+    <parent link="body"/>
+    <child link="camera_link"/>
+  </joint>
+  <!-- Camera -->
+  <link name="camera_link">
+    <collision>
+      <origin rpy="0 0 0" xyz="0 0 0"/>
+      <geometry>
+        <box size="0.05 0.05 0.05"/>
+      </geometry>
+    </collision>
+    <visual>
+      <origin rpy="0 0 0" xyz="0 0 0"/>
+      <geometry>
+        <box size="0.05 0.05 0.05"/>
+      </geometry>
+      <material name="red"/>
+    </visual>
+    <inertial>
+      <mass value="1e-5"/>
+      <origin rpy="0 0 0" xyz="0 0 0"/>
+      <inertia ixx="1e-6" ixy="0" ixz="0" iyy="1e-6" iyz="0" izz="1e-6"/>
+    </inertial>
+  </link>
+  <!-- generate an optical frame http://www.ros.org/reps/rep-0103.html#suffix-frames
+        so that ros and opencv can operate on the camera frame correctly -->
+  <joint name="camera_optical_joint" type="fixed">
+    <!-- these values have to be these values otherwise the gazebo camera image
+            won't be aligned properly with the frame it is supposedly originating from -->
+    <origin rpy="-1.57079632679 0 -1.57079632679" xyz="0 0 0"/>
+    <parent link="camera_link"/>
+    <child link="camera_link_optical"/>
+  </joint>
+  <link name="camera_link_optical">
+    </link>
   <!-- for more info visit: http://wiki.ros.org/urdf/Tutorials -->
   <link name="base_link"/>

File: config/robot/urdf/ardent_quad.xacro (robot description, xacro)
@@ -2,4 +2,5 @@
 <robot name="ardent" xmlns:xacro="http://www.ros.org/wiki/xacro">
   <xacro:include filename="$(find ardent_description)/config/robot/urdf/ardent_urdf_quad.xacro"/>
+  <xacro:include filename="$(find ardent_description)/config/robot/urdf/camera.xacro"/>
   <!-- for more info visit: http://wiki.ros.org/urdf/Tutorials -->
   <link name="base_link"/>

File: config/robot/urdf/ardent_urdf_quad.xacro (robot description, xacro)
@@ -8,4 +8,5 @@
 <!-- <xacro:property name="joint_effort" value ="10000"/>
 <xacro:property name="joint_velocity" value ="100"/> -->
+<xacro:property name="camera_link" value="0.05" />  <!-- Size of square 'camera' box -->
 <xacro:macro name="ardent" params="parent *origin">
     <joint name="j_ardent_attachment" type="fixed">

Commit message: Fixed camera

File: config/robot/urdf/ardent.urdf.xacro (robot description, xacro)
@@ -5,5 +5,6 @@
 <!-- =================================================================================== -->
 <robot name="ardent" xmlns:xacro="http://www.ros.org/wiki/xacro">
-  <!-- Size of square 'camera' box -->
+  <!-- <xacro:property name="joint_effort" value ="10000"/>
+<xacro:property name="joint_velocity" value ="100"/> -->
   <!-- Link-->
   <joint name="camera_joint" type="fixed">
@@ -45,4 +46,52 @@
   <link name="camera_link_optical">
     </link>
+  <!-- camera -->
+  <gazebo reference="camera_link">
+    <sensor name="camera1" type="camera">
+      <update_rate>30.0</update_rate>
+      <camera name="head">
+        <horizontal_fov>1.3962634</horizontal_fov>
+        <image>
+          <width>800</width>
+          <height>800</height>
+          <format>R8G8B8</format>
+        </image>
+        <clip>
+          <near>0.02</near>
+          <far>300</far>
+        </clip>
+        <noise>
+          <type>gaussian</type>
+          <!-- Noise is sampled independently per pixel on each frame.
+                That pixel's noise value is added to each of its color
+                channels, which at that point lie in the range [0,1]. -->
+          <mean>0.0</mean>
+          <stddev>0.007</stddev>
+        </noise>
+      </camera>
+      <!-- Depth Plugin -->
+      <plugin filename="libgazebo_ros_camera.so" name="camera_controller">
+        <alwaysOn>true</alwaysOn>
+        <updateRate>0.0</updateRate>
+        <cameraName>rrbot/camera1</cameraName>
+        <imageTopicName>image_raw</imageTopicName>
+        <cameraInfoTopicName>camera_info</cameraInfoTopicName>
+        <frameName>camera_link_optical</frameName>
+        <!-- setting hackBaseline to anything but 0.0 will cause a misalignment
+                between the gazebo sensor image and the frame it is supposed to
+                be attached to -->
+        <hackBaseline>0.0</hackBaseline>
+        <distortionK1>0.0</distortionK1>
+        <distortionK2>0.0</distortionK2>
+        <distortionK3>0.0</distortionK3>
+        <distortionT1>0.0</distortionT1>
+        <distortionT2>0.0</distortionT2>
+        <CxPrime>0</CxPrime>
+        <Cx>0.0</Cx>
+        <Cy>0.0</Cy>
+        <focalLength>0.0</focalLength>
+      </plugin>
+    </sensor>
+  </gazebo>
   <!-- for more info visit: http://wiki.ros.org/urdf/Tutorials -->
   <link name="base_link"/>
@@ -169,8 +218,8 @@
     </inertial>
     <visual>
-      <origin rpy="0 1.57 0" xyz="0.075 0 0"/>
+      <origin rpy="0 1.57 0" xyz="0.125 0 0"/>
       <geometry>
         <!-- <box size="0.022 0.25 0.0325" /> -->
-        <cylinder length="0.15" radius="0.015"/>
+        <cylinder length="0.25" radius="0.015"/>
         <!--<mesh filename="package://phantomx_description/meshes/thigh_l.STL"  scale="1 1 1"/>-->
       </geometry>
@@ -180,7 +229,7 @@
     </visual>
     <collision>
-      <origin rpy="0 1.57 0" xyz="0.075 0 0"/>
-      <geometry>
-        <cylinder length="0.15" radius="0.015"/>
+      <origin rpy="0 1.57 0" xyz="0.125 0 0"/>
+      <geometry>
+        <cylinder length="0.25" radius="0.015"/>
         <!-- <mesh filename="package://phantomx_description/meshes/thigh_l_coll.STL"  scale="1 1 1"/> -->
       </geometry>
@@ -264,5 +313,5 @@
     <parent link="femur_1"/>
     <child link="tibia_1"/>
-    <origin rpy="0 0 0" xyz="0.125 0 0"/>
+    <origin rpy="0 0 0" xyz="0.25 0 0"/>
     <axis xyz="0 0 1"/>
     <limit effort="30" lower="-3.14" upper="3.14" velocity="0.5"/>
@@ -421,8 +470,8 @@
     </inertial>
     <visual>
-      <origin rpy="0 1.57 0" xyz="0.075 0 0"/>
+      <origin rpy="0 1.57 0" xyz="0.125 0 0"/>
       <geometry>
         <!-- <box size="0.022 0.25 0.0325" /> -->
-        <cylinder length="0.15" radius="0.015"/>
+        <cylinder length="0.25" radius="0.015"/>
         <!--<mesh filename="package://phantomx_description/meshes/thigh_l.STL"  scale="1 1 1"/>-->
       </geometry>
@@ -432,7 +481,7 @@
     </visual>
     <collision>
-      <origin rpy="0 1.57 0" xyz="0.075 0 0"/>
-      <geometry>
-        <cylinder length="0.15" radius="0.015"/>
+      <origin rpy="0 1.57 0" xyz="0.125 0 0"/>
+      <geometry>
+        <cylinder length="0.25" radius="0.015"/>
         <!-- <mesh filename="package://phantomx_description/meshes/thigh_l_coll.STL"  scale="1 1 1"/> -->
       </geometry>
@@ -516,5 +565,5 @@
     <parent link="femur_2"/>
     <child link="tibia_2"/>
-    <origin rpy="0 0 0" xyz="0.125 0 0"/>
+    <origin rpy="0 0 0" xyz="0.25 0 0"/>
     <axis xyz="0 0 1"/>
     <limit effort="30" lower="-3.14" upper="3.14" velocity="0.5"/>
@@ -673,8 +722,8 @@
     </inertial>
     <visual>
-      <origin rpy="0 1.57 0" xyz="0.075 0 0"/>
+      <origin rpy="0 1.57 0" xyz="0.125 0 0"/>
       <geometry>
         <!-- <box size="0.022 0.25 0.0325" /> -->
-        <cylinder length="0.15" radius="0.015"/>
+        <cylinder length="0.25" radius="0.015"/>
         <!--<mesh filename="package://phantomx_description/meshes/thigh_l.STL"  scale="1 1 1"/>-->
       </geometry>
@@ -684,7 +733,7 @@
     </visual>
     <collision>
-      <origin rpy="0 1.57 0" xyz="0.075 0 0"/>
-      <geometry>
-        <cylinder length="0.15" radius="0.015"/>
+      <origin rpy="0 1.57 0" xyz="0.125 0 0"/>
+      <geometry>
+        <cylinder length="0.25" radius="0.015"/>
         <!-- <mesh filename="package://phantomx_description/meshes/thigh_l_coll.STL"  scale="1 1 1"/> -->
       </geometry>
@@ -768,5 +817,5 @@
     <parent link="femur_3"/>
     <child link="tibia_3"/>
-    <origin rpy="0 0 0" xyz="0.125 0 0"/>
+    <origin rpy="0 0 0" xyz="0.25 0 0"/>
     <axis xyz="0 0 1"/>
     <limit effort="30" lower="-3.14" upper="3.14" velocity="0.5"/>
@@ -925,8 +974,8 @@
     </inertial>
     <visual>
-      <origin rpy="0 1.57 0" xyz="0.075 0 0"/>
+      <origin rpy="0 1.57 0" xyz="0.125 0 0"/>
       <geometry>
         <!-- <box size="0.022 0.25 0.0325" /> -->
-        <cylinder length="0.15" radius="0.015"/>
+        <cylinder length="0.25" radius="0.015"/>
         <!--<mesh filename="package://phantomx_description/meshes/thigh_l.STL"  scale="1 1 1"/>-->
       </geometry>
@@ -936,7 +985,7 @@
     </visual>
     <collision>
-      <origin rpy="0 1.57 0" xyz="0.075 0 0"/>
-      <geometry>
-        <cylinder length="0.15" radius="0.015"/>
+      <origin rpy="0 1.57 0" xyz="0.125 0 0"/>
+      <geometry>
+        <cylinder length="0.25" radius="0.015"/>
         <!-- <mesh filename="package://phantomx_description/meshes/thigh_l_coll.STL"  scale="1 1 1"/> -->
       </geometry>
@@ -1020,5 +1069,5 @@
     <parent link="femur_4"/>
     <child link="tibia_4"/>
-    <origin rpy="0 0 0" xyz="0.125 0 0"/>
+    <origin rpy="0 0 0" xyz="0.25 0 0"/>
     <axis xyz="0 0 1"/>
     <limit effort="30" lower="-3.14" upper="3.14" velocity="0.5"/>

File: config/robot/urdf/ardent_urdf_quad.xacro (robot description, xacro)
@@ -8,5 +8,4 @@
 <!-- <xacro:property name="joint_effort" value ="10000"/>
 <xacro:property name="joint_velocity" value ="100"/> -->
-<xacro:property name="camera_link" value="0.05" />  <!-- Size of square 'camera' box -->
 <xacro:macro name="ardent" params="parent *origin">
     <joint name="j_ardent_attachment" type="fixed">
@@ -139,8 +138,8 @@
     </inertial>
     <visual>
-      <origin xyz="0.075 0 0" rpy="0 1.57 0"  />
+      <origin xyz="0.125 0 0" rpy="0 1.57 0"  />
       <geometry>
         <!-- <box size="0.022 0.25 0.0325" /> -->
-        <cylinder  radius="0.015" length="0.15" />
+        <cylinder  radius="0.015" length="0.25" />
         <!--<mesh filename="package://phantomx_description/meshes/thigh_l.STL"  scale="1 1 1"/>-->
       </geometry>
@@ -150,7 +149,7 @@
     </visual>
     <collision>
-      <origin xyz="0.075 0 0" rpy="0 1.57 0"  />
-      <geometry>
-        <cylinder  radius="0.015" length="0.15" />
+      <origin xyz="0.125 0 0" rpy="0 1.57 0"  />
+      <geometry>
+        <cylinder  radius="0.015" length="0.25" />
         <!-- <mesh filename="package://phantomx_description/meshes/thigh_l_coll.STL"  scale="1 1 1"/> -->
       </geometry>
@@ -234,5 +233,5 @@
     <parent link="femur_${suffix}"/>
     <child link="tibia_${suffix}"/>
-    <origin xyz="0.125 0 0" rpy="0 0 0" />
+    <origin xyz="0.25 0 0" rpy="0 0 0" />
     <axis xyz="0 0 1" />
     <limit effort="30" velocity="0.5" lower="-3.14" upper="3.14" />

File: config/robot/urdf/camera.xacro (robot description, xacro)
@@ -43,3 +43,51 @@
     <link name="camera_link_optical">
     </link>
+    <!-- camera -->
+    <gazebo reference="camera_link">
+        <sensor type="camera" name="camera1">
+        <update_rate>30.0</update_rate>
+        <camera name="head">
+            <horizontal_fov>1.3962634</horizontal_fov>
+            <image>
+            <width>800</width>
+            <height>800</height>
+            <format>R8G8B8</format>
+            </image>
+            <clip>
+            <near>0.02</near>
+            <far>300</far>
+            </clip>
+            <noise>
+            <type>gaussian</type>
+            <!-- Noise is sampled independently per pixel on each frame.
+                That pixel's noise value is added to each of its color
+                channels, which at that point lie in the range [0,1]. -->
+            <mean>0.0</mean>
+            <stddev>0.007</stddev>
+            </noise>
+        </camera>
+    <!-- Depth Plugin -->
+        <plugin name="camera_controller" filename="libgazebo_ros_camera.so">
+            <alwaysOn>true</alwaysOn>
+            <updateRate>0.0</updateRate>
+            <cameraName>rrbot/camera1</cameraName>
+            <imageTopicName>image_raw</imageTopicName>
+            <cameraInfoTopicName>camera_info</cameraInfoTopicName>
+            <frameName>camera_link_optical</frameName>
+            <!-- setting hackBaseline to anything but 0.0 will cause a misalignment
+                between the gazebo sensor image and the frame it is supposed to
+                be attached to -->
+            <hackBaseline>0.0</hackBaseline>
+            <distortionK1>0.0</distortionK1>
+            <distortionK2>0.0</distortionK2>
+            <distortionK3>0.0</distortionK3>
+            <distortionT1>0.0</distortionT1>
+            <distortionT2>0.0</distortionT2>
+            <CxPrime>0</CxPrime>
+            <Cx>0.0</Cx>
+            <Cy>0.0</Cy>
+            <focalLength>0.0</focalLength>
+        </plugin>
+        </sensor>
+    </gazebo>
 </robot>
